File: pcb/phone/main.kicad_sch (KiCad schematic)
At the start: 0 parts

Commit message: Align docs to MPCIe modem plan: flat sheet + global labels
Rewrite MCU<->Modem Link section in block-diagram.md for MPCIe variant:
- 8 signals fit exactly one TXB0108 (6 UART + RST + STATUS), no second
  shifter needed (LGA needs 10+ with PWRKEY + DCD)
- No PWRKEY on MPCIe edge connector (auto-powers on VCC, TBD with Techship)
- WAKE# (pin 1) is a falling-edge interrupt, not a level-ready signal like
  LGA STATUS (pin 49) -- different semantics documented
- Global label naming convention: MODEM_* (1.8V side), MCU_* (3.3V side),
  PCM_* (modem<->codec), USIM_* (modem<->SIM), MODEM_USB_* (modem USB)

Fix USB naming conflict: modem USB renamed from USB_DP/USB_DN to
MODEM_USB_DP/MODEM_USB_DN to avoid collision with MCU USB labels already
in the power schematic.

Fix MPCIe power: VCC pins use +3.3V (not +BATT -- raw LiPo would damage
the 3.3V-only card). LGA-only labels (MODEM_PWRKEY, GNSS_ANT, MAIN_ANT)
marked as not-placed in MPCIe wiring.

Remove hierarchical sheet references throughout modem section (flat sheet
+ global labels, not sub-sheets). Delete modem_lga.kicad_sch and
modem_mpcie.kicad_sch (hierarchical sub-sheets no longer used).

Update AGENTS.md, README.md, constraints.md, requirements.md, bom.md,
reference/README.md to reflect MPCIe as primary form factor (not "under
evaluation"), flat sheet approach, and SIM socket correction (not onboard).

Generated with [Devin](https://devin.ai)

Co-Authored-By: Devin <158243242+devin-ai-integration[bot]@users.noreply.github.com>
Other:
- removed sheet modem_lga
- removed sheet modem_mpcie
