File: pcb/phone/phone.kicad_sch (KiCad schematic)
At the start: 0 parts

Commit message: Build power schematic + lock power IC pinouts/wiring
Power section of phone.kicad_sch: USB-C (J1), MCP73831 charger (U6),
TPS63021 buck-boost (U4), TPS7A02 LDO (U5), MAX17048 fuel gauge (U7),
USBLC6-2 ESD (U10), J_BATT battery connector, STAT LED, passives.

Documented pinouts/wiring for J1, U4, U5, U6, U7, U10 in block-diagram.md.
Locked J_BATT = JST S2B-PH-SM4-TB (C295747). Resolved all power open
questions: PG to MCU (EXTI + 10k pullup to +3.3V), TPS7A02 EN tie to IN,
ALRT to MCU (EXTI + 10k pullup), I2C no conflict (MAX17048=0x36,
ALC5651=0x1A), R_PROG=2k (500mA = 0.42C on 1200mAh), STAT=LED+470R.

Corrections verified against datasheets: MAX17048 pinout (6 of 8 pins were
wrong in docs, VDD moved to +BATT), MCP73831 SOT-23-5 to DFN-8 package,
USBLC6-2 protects VBUS (pin 5, not just D+/D-), MCP73831 STAT behavior
inverted in docs (LED circuit was correct), net names standardized
(+BATT/+3.3V/+1V8), ref designators renamed in schematic (USBC1 to J1,
CN1 to J_BATT, D1 to U10).

Datasheets downloaded + indexed: max17048.pdf, mcp73831.pdf, usblc6-2.pdf.
New project rule: datasheets must be downloaded before citing specs
(added to AGENTS.md + docs/reference/README.md).

New KiCad library parts: J_BATT footprint + 3D, R0603 footprint + 3D,
L0603 (ferrite bead) footprint + 3D. C0805 footprint LCSC part updated
to C77074 (22uF) and 3D path made relative.

.gitignore: add *.kicad_prl (KiCad user-local project rules).

Generated with [Devin](https://devin.ai)

Co-Authored-By: Devin <158243242+devin-ai-integration[bot]@users.noreply.github.com>
Parts:
- added C1, C7: CC0603KRX7R9BB104, easyeda2kicad:C0603, symbol easyeda2kicad:CC0603KRX7R9BB104
- added C10, C11: GRM188R61C475KE11D, easyeda2kicad:C0603, symbol easyeda2kicad:GRM188R61C475KE11D
- added C2, C3: GRM21BR61H106KE43L, easyeda2kicad:C0805, symbol easyeda2kicad:GRM21BR61H106KE43L
- added C4, C5, C6: GRM21BR61A226ME51L, easyeda2kicad:C0805, symbol easyeda2kicad:GRM21BR61A226ME51L
- added C8, C9: GRM188R61C105KA93D, easyeda2kicad:C0603, symbol easyeda2kicad:GRM188R61C105KA93D
- added CN1: S2B-PH-SM4-TB, easyeda2kicad:CONN-SMD_P2.00_S2B-PH-SM4-TB-LF-SN, symbol easyeda2kicad:S2B-PH-SM4-TB
- added D1: USBLC6-2SC6, easyeda2kicad:SOT-23-6_L2.9-W1.6-P0.95-LS2.8-BL, symbol easyeda2kicad:USBLC6-2SC6
- added L1: XFL4020-152MEC, easyeda2kicad:IND-SMD_L4.0-W4.0-A, symbol easyeda2kicad:XFL4020-152MEC
- added LED1: LTST-C191TBKT, easyeda2kicad:LED0603-RD, symbol easyeda2kicad:LTST-C191TBKT
- added R1: RC0603JR-071ML, easyeda2kicad:R0603, symbol easyeda2kicad:RC0603JR-071ML
- added R2, R4: RC0603JR-0710KL, easyeda2kicad:R0603, symbol easyeda2kicad:RC0603JR-0710KL
- added R3: RC0603JR-07470RL, easyeda2kicad:R0603, symbol easyeda2kicad:RC0603JR-07470RL
- added R5: RC0603FR-072KL, easyeda2kicad:R0603, symbol easyeda2kicad:RC0603FR-072KL
- added R6, R7: RC0603FR-075K1L, easyeda2kicad:R0603, symbol easyeda2kicad:RC0603FR-075K1L
- added U4: TPS63021DSJR, easyeda2kicad:VSON-14_L4.0-W3.0-P0.50-BL-EP_TI_DSJ, symbol easyeda2kicad:TPS63021DSJR
- added U5: TPS7A0218PDBVR, easyeda2kicad:SOT-23-5_L2.9-W1.6-P0.95-LS2.8-BL, symbol easyeda2kicad:TPS7A0218PDBVR
- added U6: MCP73831-2ACI/MC, easyeda2kicad:TDFN-8_L3.0-W2.0-P0.50-BL-EP1.6, symbol easyeda2kicad:MCP73831-2ACI_MC
- added U7: MAX17048G+T10, easyeda2kicad:TDFN-8_L2.0-W2.0-P0.50-BL-EP1.2, symbol easyeda2kicad:MAX17048G+T10
- added USBC1: TYPE-C-31-M-12, easyeda2kicad:USB-C_SMD-TYPE-C-31-M-12_1, symbol easyeda2kicad:TYPE-C-31-M-12
Connections:
- new net: R6.2, USBC1.A5 (CC1)
- new net: R7.2, USBC1.B5 (CC2)
- new net: L1.1, U4.8 (L1), U4.9 (L1)
- new net: L1.2, U4.6 (L2), U4.7 (L2)
- new net: LED1.1 (-), U6.5 (STAT)
- new net: LED1.2 (+), R3.1
- new net: C1.2, U4.1 (VINA)
- new net: R1.2, U4.12 (EN)
- new net: R5.2, U6.8 (PROG)
- new net +1V8: C9.2, U5.5 (OUT)
- new net +3.3V: C4.2, C5.2, C6.2, C8.2, R2.2, R4.1, U4.3 (FB), U4.4 (VOUT), U4.5 (VOUT), U5.1 (IN), U5.3 (EN)
- new net +BATT: C10.2, C2.1, C3.1, C7.2, CN1.1, R1.1, U4.10 (VIN), U4.11 (VIN), U6.3 (VBAT), U6.4 (VBAT), U7.2 (CELL), U7.3 (VDD)
- new net 3V3_OK: R4.2, U4.14 (PG)
- new net FUEL_ALERT: R2.1, U7.5 (~{ALRT})
- new net GND: C1.1, C10.1, C11.2, C2.2, C3.2, C4.1, C5.1, C6.1, C7.1, C8.1, C9.1, CN1.2, CN1.3, CN1.4, D1.2, R5.1, R6.1, R7.1, U4.13 (PS/SYNC), U4.15 (PGND), U4.2 (GND), U5.2 (GND), U6.6 (VSS), U6.9 (EP), U7.1 (CTG), U7.4 (GND), U7.6 (QSTRT), U7.9 (EP), USBC1.1 (EH), USBC1.2 (EH), USBC1.3 (EH), USBC1.4 (EH), USBC1.A1B12 (GND), USBC1.A8 (SBU1), USBC1.B1A12 (GND), USBC1.B8 (SBU2)
- new net I2C_SCL: U7.7 (SCL)
- new net I2C_SDA: U7.8 (SDA)
- new net USB_DN: D1.3, D1.4, USBC1.A7 (DN1), USBC1.B7 (DN2)
- new net USB_DP: D1.1, D1.6, USBC1.A6 (DP1), USBC1.B6 (DP2)
- new net VBUS: C11.1, D1.5, R3.2, U6.1 (VDD), U6.2 (VDD), USBC1.A4B9 (VBUS), USBC1.B4A9 (VBUS)
Other:
- note added: "DONE: NEEDS REVIEW"
- note added: "I2C LINES NEED PULLUP AT MCU"

Commit message: Update schematic refs to new lib names + remove old library files
- Update phone.kicad_sch: 46 symbol references changed from
  easyeda2kicad:SYMBOL to passives:/ics:/connectors:SYMBOL
  (19 unique symbols, both lib_id and symbol declarations)
- Remove easyeda2kicad.kicad_sym (superseded by 4 split libraries)
- Remove missing_parts.kicad_sym (merged into split libraries)
- Remove superseded MAX9880A footprints (footprints.pretty/ — not tracked,
  removed from disk; MAX9880A was SUPERSEDED 2026-07-19 by ALC5651)
- Remove superseded ultralibrarian.kicad_sym (MAX9880A symbol — not tracked,
  removed from disk)

Generated with [Devin](https://devin.ai)

Co-Authored-By: Devin <158243242+devin-ai-integration[bot]@users.noreply.github.com>
Parts:
- C1, C7: symbol easyeda2kicad:CC0603KRX7R9BB104 -> passives:CC0603KRX7R9BB104
- C10, C11: symbol easyeda2kicad:GRM188R61C475KE11D -> passives:GRM188R61C475KE11D
- C2, C3: symbol easyeda2kicad:GRM21BR61H106KE43L -> passives:GRM21BR61H106KE43L
- C4, C5, C6: symbol easyeda2kicad:GRM21BR61A226ME51L -> passives:GRM21BR61A226ME51L
- C8, C9: symbol easyeda2kicad:GRM188R61C105KA93D -> passives:GRM188R61C105KA93D
- CN1: symbol easyeda2kicad:S2B-PH-SM4-TB -> connectors:S2B-PH-SM4-TB
- D1: symbol easyeda2kicad:USBLC6-2SC6 -> ics:USBLC6-2SC6
- L1: symbol easyeda2kicad:XFL4020-152MEC -> passives:XFL4020-152MEC
- LED1: symbol easyeda2kicad:LTST-C191TBKT -> passives:LTST-C191TBKT
- R1: symbol easyeda2kicad:RC0603JR-071ML -> passives:RC0603JR-071ML
- R2, R4: symbol easyeda2kicad:RC0603JR-0710KL -> passives:RC0603JR-0710KL
- R3: symbol easyeda2kicad:RC0603JR-07470RL -> passives:RC0603JR-07470RL
- R5: symbol easyeda2kicad:RC0603FR-072KL -> passives:RC0603FR-072KL
- R6, R7: symbol easyeda2kicad:RC0603FR-075K1L -> passives:RC0603FR-075K1L
- U4: symbol easyeda2kicad:TPS63021DSJR -> ics:TPS63021DSJR
- U5: symbol easyeda2kicad:TPS7A0218PDBVR -> ics:TPS7A0218PDBVR
- U6: symbol easyeda2kicad:MCP73831-2ACI_MC -> ics:MCP73831-2ACI_MC
- U7: symbol easyeda2kicad:MAX17048G+T10 -> ics:MAX17048G+T10
- USBC1: symbol easyeda2kicad:TYPE-C-31-M-12 -> connectors:TYPE-C-31-M-12
Changed lines of the file:
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@@
 	)
 	(symbol
-		(lib_id "easyeda2kicad:TYPE-C-31-M-12")
+		(lib_id "connectors:TYPE-C-31-M-12")
 		(at 172.72 129.54 0)
 		(mirror y)
@@
 	)
 	(symbol
-		(lib_id "easyeda2kicad:MAX17048G+T10")
+		(lib_id "ics:MAX17048G+T10")
 		(at 69.85 101.6 0)
 		(unit 1)
@@
 	(symbol
 		(lib_name "CC0603KRX7R9BB104_1")
-		(lib_id "easyeda2kicad:CC0603KRX7R9BB104")
+		(lib_id "passives:CC0603KRX7R9BB104")
 		(at 49.53 109.22 90)
 		(unit 1)
@@
 	)
 	(symbol
-		(lib_id "easyeda2kicad:S2B-PH-SM4-TB")
+		(lib_id "connectors:S2B-PH-SM4-TB")
 		(at 40.64 35.56 180)
 		(unit 1)
@@
 	)
 	(symbol
-		(lib_id "easyeda2kicad:RC0603JR-0710KL")
+		(lib_id "passives:RC0603JR-0710KL")
 		(at 86.36 49.53 90)
 		(unit 1)
@@
 	)
 	(symbol
-		(lib_id "easyeda2kicad:RC0603FR-075K1L")
+		(lib_id "passives:RC0603FR-075K1L")
 		(at 190.5 123.19 0)
 		(mirror y)
@@
 	)
 	(symbol
-		(lib_id "easyeda2kicad:GRM21BR61A226ME51L")
+		(lib_id "passives:GRM21BR61A226ME51L")
 		(at 129.54 39.37 90)
 		(unit 1)
@@
 	)
 	(symbol
-		(lib_id "easyeda2kicad:RC0603FR-075K1L")
+		(lib_id "passives:RC0603FR-075K1L")
 		(at 190.5 138.43 0)
 		(mirror y)
@@
 	)
 	(symbol
-		(lib_id "easyeda2kicad:XFL4020-152MEC")
+		(lib_id "passives:XFL4020-152MEC")
 		(at 104.14 17.78 0)
 		(unit 1)
@@
 	)
 	(symbol
-		(lib_id "easyeda2kicad:LTST-C191TBKT")
+		(lib_id "passives:LTST-C191TBKT")
 		(at 46.99 162.56 180)
 		(unit 1)
@@
 	)
 	(symbol
-		(lib_id "easyeda2kicad:TPS63021DSJR")
+		(lib_id "ics:TPS63021DSJR")
 		(at 104.14 39.37 180)
 		(unit 1)
@@
 	)
 	(symbol
-		(lib_id "easyeda2kicad:RC0603FR-072KL")
+		(lib_id "passives:RC0603FR-072KL")
 		(at 87.63 161.29 180)
 		(unit 1)
@@
 	)
 	(symbol
-		(lib_id "easyeda2kicad:GRM21BR61A226ME51L")
+		(lib_id "passives:GRM21BR61A226ME51L")
 		(at 142.24 39.37 90)
 		(unit 1)
@@
 	)
 	(symbol
-		(lib_id "easyeda2kicad:GRM21BR61A226ME51L")
+		(lib_id "passives:GRM21BR61A226ME51L")
 		(at 135.89 39.37 90)
 		(unit 1)
@@
 	)
 	(symbol
-		(lib_id "easyeda2kicad:CC0603KRX7R9BB104")
+		(lib_id "passives:CC0603KRX7R9BB104")
 		(at 119.38 49.53 270)
 		(mirror x)
@@
 	)
 	(symbol
-		(lib_id "easyeda2kicad:GRM188R61C475KE11D")
+		(lib_id "passives:GRM188R61C475KE11D")
 		(at 25.4 158.75 270)
 		(unit 1)
@@
 	)
 	(symbol
-		(lib_id "easyeda2kicad:GRM188R61C475KE11D")
+		(lib_id "passives:GRM188R61C475KE11D")
 		(at 90.17 153.67 180)
 		(unit 1)
@@
 	)
 	(symbol
-		(lib_id "easyeda2kicad:GRM21BR61H106KE43L")
+		(lib_id "passives:GRM21BR61H106KE43L")
 		(at 62.23 39.37 270)
 		(unit 1)
@@
 	)
 	(symbol
-		(lib_id "easyeda2kicad:TPS7A0218PDBVR")
+		(lib_id "ics:TPS7A0218PDBVR")
 		(at 185.42 39.37 0)
 		(unit 1)
@@
 	)
 	(symbol
-		(lib_id "easyeda2kicad:GRM188R61C105KA93D")
+		(lib_id "passives:GRM188R61C105KA93D")
 		(at 199.39 44.45 90)
 		(unit 1)
@@
 	)
 	(symbol
-		(lib_id "easyeda2kicad:MCP73831-2ACI_MC")
+		(lib_id "ics:MCP73831-2ACI_MC")
 		(at 67.31 161.29 0)
 		(unit 1)
@@
 	)
 	(symbol
-		(lib_id "easyeda2kicad:GRM21BR61H106KE43L")
+		(lib_id "passives:GRM21BR61H106KE43L")
 		(at 71.12 39.37 270)
 		(unit 1)
@@
 	)
 	(symbol
-		(lib_id "easyeda2kicad:RC0603JR-071ML")
+		(lib_id "passives:RC0603JR-071ML")
 		(at 81.28 39.37 0)
 		(unit 1)
@@
 	)
 	(symbol
-		(lib_id "easyeda2kicad:GRM188R61C105KA93D")
+		(lib_id "passives:GRM188R61C105KA93D")
 		(at 170.18 41.91 90)
 		(unit 1)
@@
 	)
 	(symbol
-		(lib_id "easyeda2kicad:RC0603JR-07470RL")
+		(lib_id "passives:RC0603JR-07470RL")
 		(at 36.83 161.29 180)
 		(unit 1)
@@
 	)
 	(symbol
-		(lib_id "easyeda2kicad:RC0603JR-0710KL")
+		(lib_id "passives:RC0603JR-0710KL")
 		(at 106.68 101.6 90)
 		(unit 1)
@@
 	)
 	(symbol
-		(lib_id "easyeda2kicad:USBLC6-2SC6")
+		(lib_id "ics:USBLC6-2SC6")
 		(at 243.84 130.81 0)
 		(unit 1)

Commit message: WIP: mPCIe vs LGA modem exploration + connectors.kicad_sym encoding break
Adds Mini PCIe connector (PCIE-52P40H_C444926) and footprint, plus
modem_mpcie.kicad_sch / modem_lga.kicad_sch sheets to compare the two
modem mounting options. Docs updated for the evaluation.

NOTE: pcb/phone/lib/connectors.kicad_sym is currently broken -- a UTF-8
BOM was prepended and all CJK strings got CP1252-mojibake'd (likely by
a Windows editor saving the file). KiCad loads the library as empty
because the S-expression parser chokes on the BOM before the opening
paren. This commit preserves the broken state as a checkpoint; the
encoding will be repaired in a follow-up commit.

Generated with [Devin](https://devin.ai)

Co-Authored-By: Devin <158243242+devin-ai-integration[bot]@users.noreply.github.com>
Parts:
- C7: Manufacturer YAGEO(ÃƒÆ’Ã†â€™Ãƒâ€šÃ‚Â¥ÃƒÆ’Ã‚Â¢ÃƒÂ¢Ã¢â‚¬Å¡Ã‚Â¬Ãƒâ€šÃ‚ÂºÃƒÆ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 -> YAGEO(国巨)
- LED1: Manufacturer LITEON(光宝科技) -> LITEON(光宝)
Changed lines of the file:
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@@
 			)
 		)
-		(property "Description" ""
+		(property "Description" "USB-C 16-pin 2.0 receptacle"
 			(at 172.72 129.54 0)
 			(hide yes)
@@
 			)
 		)
-		(property "Description" ""
+		(property "Description" "Fuel gauge I2C TDFN-8"
 			(at 69.85 101.6 0)
 			(hide yes)
@@
 	)
 	(symbol
-		(lib_name "CC0603KRX7R9BB104_1")
 		(lib_id "passives:CC0603KRX7R9BB104")
 		(at 49.53 109.22 90)
@@
 			)
 		)
-		(property "Description" "100nF 0603 cap"
+		(property "Description" "100nF (104) ±10% 50V"
 			(at 49.53 109.22 0)
 			(hide yes)
@@
 			)
 		)
-		(property "Manufacturer" "YAGEO(ÃƒÆ’Ã†â€™Ãƒâ€šÃ‚Â¥ÃƒÆ’Ã‚Â¢ÃƒÂ¢Ã¢â‚¬Å¡Ã‚Â¬Ãƒâ€šÃ‚ÂºÃƒÆ’Ã¢â‚¬Å¡Ãƒâ€šÃ‚Â½ÃƒÆ’Ã†â€™Ãƒâ€šÃ‚Â¥ÃƒÆ’Ã¢â‚¬Å¡Ãƒâ€šÃ‚Â·ÃƒÆ’Ã¢â‚¬Å¡Ãƒâ€šÃ‚Â¨)"
+		(property "Manufacturer" "YAGEO(国巨)"
 			(at 62.23 109.22 0)
 			(hide yes)
@@
 			)
 		)
-		(property "Description" ""
+		(property "Description" "JST-PH 2-pin battery conn"
 			(at 40.64 35.56 0)
 			(hide yes)
@@
 			)
 		)
-		(property "Description" "10kΩ 0603 res"
+		(property "Description" "10k 5% 0603 resistor"
 			(at 86.36 49.53 0)
 			(hide yes)
@@
 			)
 		)
-		(property "Description" "5.1kΩ 0603 1% res"
+		(property "Description" "5.1k 1% 0603 resistor"
 			(at 190.5 123.19 0)
 			(hide yes)
@@
 			)
 		)
-		(property "Description" ""
+		(property "Description" "22uF 10V X5R 0805 cap"
 			(at 129.54 39.37 0)
 			(hide yes)
@@
 			)
 		)
-		(property "Description" "5.1kΩ 0603 1% res"
+		(property "Description" "5.1k 1% 0603 resistor"
 			(at 190.5 138.43 0)
 			(hide yes)
@@
 			)
 		)
-		(property "Description" ""
+		(property "Description" "1.5uH 4.4A inductor"
 			(at 104.14 17.78 0)
 			(hide yes)
@@
 			)
 		)
-		(property "Description" "Blue LED 0603"
+		(property "Description" "Blue LED 0603 468nm"
 			(at 46.99 162.56 0)
 			(hide yes)
@@
 			)
 		)
-		(property "Manufacturer" "LITEON(光宝科技)"
+		(property "Manufacturer" "LITEON(光宝)"
 			(at 46.99 148.59 0)
 			(hide yes)
@@
 			)
 		)
-		(property "Description" ""
+		(property "Description" "3.3V buck-boost 4A VSON14"
 			(at 104.14 39.37 0)
 			(hide yes)
@@
 			)
 		)
-		(property "Description" "2kΩ 0603 1% res"
+		(property "Description" "2k 1% 0603 resistor"
 			(at 87.63 161.29 0)
 			(hide yes)
@@
 			)
 		)
-		(property "Description" ""
+		(property "Description" "22uF 10V X5R 0805 cap"
 			(at 142.24 39.37 0)
 			(hide yes)
@@
 			)
 		)
-		(property "Description" ""
+		(property "Description" "22uF 10V X5R 0805 cap"
 			(at 135.89 39.37 0)
 			(hide yes)
@@
 			)
 		)
-		(property "Description" "4.7µF 0603 cap"
+		(property "Description" "4.7uF 16V X5R 0603 cap"
 			(at 25.4 158.75 0)
 			(hide yes)
@@
 			)
 		)
-		(property "Description" "4.7µF 0603 cap"
+		(property "Description" "4.7uF 16V X5R 0603 cap"
 			(at 90.17 153.67 0)
 			(hide yes)
@@
 			)
 		)
-		(property "Description" ""
+		(property "Description" "10uF 50V X5R 0805 cap"
 			(at 62.23 39.37 0)
 			(hide yes)
@@
 			)
 		)
-		(property "Description" ""
+		(property "Description" "1.8V LDO 200mA SOT23-5"
 			(at 185.42 39.37 0)
 			(hide yes)
@@
 			)
 		)
-		(property "Description" "1µF 0603 cap"
+		(property "Description" "1uF(105) ±10% 16V"
 			(at 199.39 44.45 0)
 			(hide yes)
@@
 			)
 		)
-		(property "Description" ""
+		(property "Description" "LiPo charger 500mA"
 			(at 67.31 161.29 0)
 			(hide yes)
@@
 			)
 		)
-		(property "Description" ""
+		(property "Description" "10uF 50V X5R 0805 cap"
 			(at 71.12 39.37 0)
 			(hide yes)
@@
 			)
 		)
-		(property "Description" ""
+		(property "Description" "1M 5% 0603 resistor"
 			(at 81.28 39.37 0)
 			(hide yes)
@@
 			)
 		)
-		(property "Description" "1µF 0603 cap"
+		(property "Description" "1uF(105) ±10% 16V"
 			(at 170.18 41.91 0)
 			(hide yes)
@@
 			)
 		)
-		(property "Datasheet" "https://lcsc.com/product-detail/Chip-Resistor-Surface-Mount_YAGEO-RC0603JR-07470RL_C114433.html"
+		(property "Datasheet" "https://lcsc.com/product-detail/Chip-Resistor-Surface-Mount_470R-471-5_C114433.html"
 			(at 36.83 151.13 0)
 			(hide yes)
@@
 			)
 		)
-		(property "Description" "470Ω 0603 res"
+		(property "Description" "470R 5% 0603 resistor"
 			(at 36.83 161.29 0)
 			(hide yes)
@@
 			)
 		)
-		(property "Description" "10kΩ 0603 res"
+		(property "Description" "10k 5% 0603 resistor"
 			(at 106.68 101.6 0)
 			(hide yes)
@@
 	(sheet_instances
 		(path "/"
-			(page "1")
+			(page "2")
 		)
 	)
