File: pcb/phone/phone.kicad_sch (KiCad schematic)
At the start: 27 parts, among them CN1 S2B-PH-SM4-TB, U4 TPS63021DSJR, U5 TPS7A0218PDBVR, U6 MCP73831-2ACI/MC, U7 MAX17048G+T10

Commit message: Phase 3.6-3.7: Add SIM/SD sheet with ESD protection
- sim_sd.kicad_sch: nano-SIM socket, microSD slot, 2x ESDA6V1-5SC6 ESD
  protection, decoupling caps, SIM data pull-up
- phone.kicad_sch: added SIM_SD sheet box (page 7)
- Fixed SD_CLK label to SD_CK to match MCU pin assignment

Generated with [Devin](https://devin.ai)

Co-Authored-By: Devin <158243242+devin-ai-integration[bot]@users.noreply.github.com>
Other:
- added sheet SIM_SD (sim_sd.kicad_sch)
Changed lines of the file:
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@@
+		)
+	)
+	(sheet
+		(at 254 300)
+		(size 30.48 20.32)
+		(exclude_from_sim no)
+		(in_bom yes)
+		(on_board yes)
+		(dnp no)
+		(fields_autoplaced yes)
+		(stroke
+			(width 0.1524)
+			(type solid)
+		)
+		(fill
+			(color 0 0 0 0)
+		)
+		(property "Sheetname" "SIM_SD"
+			(at 254 299 0)
+			(show_name no)
+			(do_not_autoplace no)
+			(effects
+				(font
+					(size 1.27 1.27)
+				)
+				(justify left bottom)
+			)
+		)
+		(property "Sheetfile" "sim_sd.kicad_sch"
+			(at 254 321 0)
+			(show_name no)
+			(do_not_autoplace no)
+			(effects
+				(font
+					(size 1.27 1.27)
+				)
+				(justify left top)
+			)
+		)
+		(instances
+			(project "phone"
+				(path "/451c3b43-1616-42cb-bf96-d436f4db82c2"
+					(page "7")
+				)
+			)
 		)
 	)
