File: pcb/phone/codec.kicad_sch (KiCad schematic)
At the start: 10 parts, among them U3 ALC5651-CG, U9 TXB0108PWR

Commit message: Cleanup: remove rejected part symbols, one-off scripts, stale datasheets
- Remove 7 rejected symbols from easyeda2kicad.kicad_sym (PJ-327C-4A,
  PJ-3250-5A, PJ-3240-5A, TYPE-C16PLC-H10.0, PJ-327A5JJ, PJ-327-P5,
  TYPEC-306DDW-ARP16) — replaced by Tensility 54-00298 and GCT USB4085-GF-A
- Delete 10 one-off inspection scripts (check_*.py, find_*.py, dump_*.py,
  extract_*.py) — keep only gen_*.py schematic generators
- Delete rejected datasheets (pj3126-5a, pj3240-5a, pj3250-5a, pj3f07-5p,
  N114 superseded display)
- Delete generated BOM/POS CSV files
- Add alps-ssss2.pdf and gct-usb4085.pdf to reference README index
- Include all schematic changes from previous sessions (SD pullups, VBUS
  divider fix, level shifter verification, codec caps, DCVDD fix)

Generated with [Devin](https://devin.ai)

Co-Authored-By: Devin <158243242+devin-ai-integration[bot]@users.noreply.github.com>
Parts:
- removed U9: TXB0108PWR, symbol ics:TXB0108PWR
- added C41, C42, C43, C44: CC0603KRX5R8BB225, easyeda2kicad:C0603, symbol passives:CC0603KRX5R8BB225
- added C45: GRM188R61C475KE11D, easyeda2kicad:C0603, symbol passives:GRM188R61C475KE11D
- added U12: SN74AXC4T774PWR, easyeda2kicad:TSSOP-16_L5.0-W4.4-P0.65-LS6.4-TL, symbol ics:SN74AXC4T774PWR
- renumbered C33 to C23, C34 to C24, C35 to C25, C36 to C26, J_MIC to J_MIC1, J_SPK to J_SPK1, R12 to R10, R13 to R11, U3 to U5
Connections:
- net +1V8: now also U5.8 (DACREF), U12.1 (DIR1), U12.16 (VCCA); no longer U5.40 (DCVDD)
- net +3.3V: now also U12.15 (VCCB)
- net GND: now also U5.20 (CPVREF), C41.1, C42.1, C45.2, U12.10 (GND), U12.2 (DIR2), U12.7 (DIR3), U12.8 (DIR4), U12.9 (~{OE})
- net I2S2_ADCDAT: now also U12.14 (B1)
- net I2S2_BCLK: now also U12.11 (B4)
- net I2S2_DACDAT: now also U12.13 (B2)
- net I2S2_LRCK: now also U12.12 (B3)
- net at U5.29 (BCLK2): now also U12.6 (A4)
- net at U5.28 (LRCK2): now also U12.5 (A3)
- net at U5.27 (DACDAT2): now also U12.4 (A2)
- net at U5.26 (ADCDAT2): now also U12.3 (A1)
- net at U5.11 (VREF): now also C45.1
- net at U5.14 (CPN2): now also C43.1
- net at U5.15 (CPP2): now also C43.2
- net at U5.16 (CPN1): now also C44.1
- net at U5.17 (CPP1): now also C44.2
- net at U5.19 (CPVPP): now also C42.2
- net at U5.22 (CPVEE): now also C41.2
- no-connect marks 28 -> 12
Other:
- moved on the sheet: J_MIC1, J_SPK1

Commit message: Assign footprints to 29 components missing footprint properties
All 28 custom-library components (passives, connectors, ICs) get footprints
from their symbol library defaults. J1 (SWD debug header) gets a standard
KiCad 2.54mm through-hole pin header footprint per user selection.

Footprints assigned:
- C18-C23: easyeda2kicad:C0805 (10uF 0805 caps)
- C24-C26: easyeda2kicad:C0603 (100nF 0603 caps)
- R6-R18: easyeda2kicad:R0603 (0603 resistors)
- J_HINGE2: easyeda2kicad:FPC-SMD_14P-P0.50_HDGC_0.5K-HX-14PWB
- J_MIC1, J_SPK1: easyeda2kicad:CONN-SMD_P2.00_S2B-PH-SM4-TB-LF-SN
- U2: easyeda2kicad:PCIE-SMD_PCIE-52P40H-1 (mini-PCIe)
- U3: easyeda2kicad:TSSOP-20_L6.5-W4.4-P0.65-LS6.4-BL (TXB0108)
- U5: easyeda2kicad:QFN-40_L5.0-W5.0-P0.40-BL-EP3.7 (ALC5651)
- J1: Connector_PinHeader_2.54mm:PinHeader_1x04_P2.54mm_Vertical (SWD)

Also includes KiCad's own metadata updates (title block, sheet ordering,
designator list normalization).

Generated with [Devin](https://devin.ai)

Co-Authored-By: Devin <158243242+devin-ai-integration[bot]@users.noreply.github.com>
Parts:
- C23: footprint (none) -> easyeda2kicad:C0805
- C24, C25, C26: footprint (none) -> easyeda2kicad:C0603
- J_MIC1, J_SPK1: footprint (none) -> easyeda2kicad:CONN-SMD_P2.00_S2B-PH-SM4-TB-LF-SN
- R10, R11: footprint (none) -> easyeda2kicad:R0603
- U5: footprint (none) -> easyeda2kicad:QFN-40_L5.0-W5.0-P0.40-BL-EP3.7
Changed lines of the file:
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@@
 			)
 		)
-		(property "Footprint" ""
+		(property "Footprint" "easyeda2kicad:C0603"
 			(at 99.06 168.91 0)
 			(hide yes)
@@
 			)
 		)
-		(property "Footprint" ""
+		(property "Footprint" "easyeda2kicad:R0603"
 			(at 198.12 80.01 0)
 			(hide yes)
@@
 			)
 		)
-		(property "Footprint" ""
+		(property "Footprint" "easyeda2kicad:R0603"
 			(at 158.75 78.74 0)
 			(hide yes)
@@
 			)
 		)
-		(property "Footprint" ""
+		(property "Footprint" "easyeda2kicad:C0805"
 			(at 83.82 168.91 0)
 			(hide yes)
@@
 			)
 		)
-		(property "Footprint" ""
+		(property "Footprint" "easyeda2kicad:C0603"
 			(at 223.52 168.91 0)
 			(hide yes)
@@
 			)
 		)
-		(property "Footprint" ""
+		(property "Footprint" "easyeda2kicad:CONN-SMD_P2.00_S2B-PH-SM4-TB-LF-SN"
 			(at 58.42 146.05 0)
 			(hide yes)
@@
 			)
 		)
-		(property "Footprint" ""
+		(property "Footprint" "easyeda2kicad:C0603"
 			(at 208.28 168.91 0)
 			(hide yes)
@@
 			)
 		)
-		(property "Footprint" ""
+		(property "Footprint" "easyeda2kicad:CONN-SMD_P2.00_S2B-PH-SM4-TB-LF-SN"
 			(at 58.42 123.19 0)
 			(hide yes)
@@
 			)
 		)
-		(property "Footprint" ""
+		(property "Footprint" "easyeda2kicad:QFN-40_L5.0-W5.0-P0.40-BL-EP3.7"
 			(at 138.43 129.54 0)
 			(hide yes)
