File: pcb/phone/display_daughter.kicad_sch (KiCad schematic)
At the start: 6 parts

Commit message: Cleanup: remove rejected part symbols, one-off scripts, stale datasheets
- Remove 7 rejected symbols from easyeda2kicad.kicad_sym (PJ-327C-4A,
  PJ-3250-5A, PJ-3240-5A, TYPE-C16PLC-H10.0, PJ-327A5JJ, PJ-327-P5,
  TYPEC-306DDW-ARP16) — replaced by Tensility 54-00298 and GCT USB4085-GF-A
- Delete 10 one-off inspection scripts (check_*.py, find_*.py, dump_*.py,
  extract_*.py) — keep only gen_*.py schematic generators
- Delete rejected datasheets (pj3126-5a, pj3240-5a, pj3250-5a, pj3f07-5p,
  N114 superseded display)
- Delete generated BOM/POS CSV files
- Add alps-ssss2.pdf and gct-usb4085.pdf to reference README index
- Include all schematic changes from previous sessions (SD pullups, VBUS
  divider fix, level shifter verification, codec caps, DCVDD fix)

Generated with [Devin](https://devin.ai)

Co-Authored-By: Devin <158243242+devin-ai-integration[bot]@users.noreply.github.com>
Parts:
- renumbered C37 to C27, J_DISP to J_DISP1, J_EARPIECE to J_EARPIECE1, R14 to R19

Commit message: Assign footprints to 29 components missing footprint properties
All 28 custom-library components (passives, connectors, ICs) get footprints
from their symbol library defaults. J1 (SWD debug header) gets a standard
KiCad 2.54mm through-hole pin header footprint per user selection.

Footprints assigned:
- C18-C23: easyeda2kicad:C0805 (10uF 0805 caps)
- C24-C26: easyeda2kicad:C0603 (100nF 0603 caps)
- R6-R18: easyeda2kicad:R0603 (0603 resistors)
- J_HINGE2: easyeda2kicad:FPC-SMD_14P-P0.50_HDGC_0.5K-HX-14PWB
- J_MIC1, J_SPK1: easyeda2kicad:CONN-SMD_P2.00_S2B-PH-SM4-TB-LF-SN
- U2: easyeda2kicad:PCIE-SMD_PCIE-52P40H-1 (mini-PCIe)
- U3: easyeda2kicad:TSSOP-20_L6.5-W4.4-P0.65-LS6.4-BL (TXB0108)
- U5: easyeda2kicad:QFN-40_L5.0-W5.0-P0.40-BL-EP3.7 (ALC5651)
- J1: Connector_PinHeader_2.54mm:PinHeader_1x04_P2.54mm_Vertical (SWD)

Also includes KiCad's own metadata updates (title block, sheet ordering,
designator list normalization).

Generated with [Devin](https://devin.ai)

Co-Authored-By: Devin <158243242+devin-ai-integration[bot]@users.noreply.github.com>
Parts:
- J_HINGE2: footprint (none) -> easyeda2kicad:FPC-SMD_14P-P0.50_HDGC_0.5K-HX-14PWB
Changed lines of the file:
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@@
 			)
 		)
-		(property "Footprint" ""
+		(property "Footprint" "easyeda2kicad:FPC-SMD_14P-P0.50_HDGC_0.5K-HX-14PWB"
 			(at 129.54 129.54 0)
 			(hide yes)

Commit message: Restructure display sheet for candybar + fix pinout + add backlight FET + power switch reversal
Display sheet (LOCKED):
- Fix J_DISP1 pinout to match HS20HS072RX datasheet (was 1/12 correct, now all 14 pins match)
- Add backlight FET circuit: Q1 (AO3400A), R20 (100ohm gate), R5 (10k pulldown), R19 moved to pin 10
- Fix R19 MPN: was 470ohm part with 4.7ohm value, swapped to RC0603JR-074R7L (correct 4.7ohm)
- Move display power from +1V8 to +3.3V (1.8V below VCC min 2.4V)
- Remove display_daughter sheet entry, J_HINGE1, J_HINGE2, OUTER_CS/OUTER_DC
- Add no-connect flags on MCU PG9/PG10 (freed from outer display)
- FPC connector orientation review flagged for PCB layout phase

Power switch (reversed 2026-08-27):
- Move SW21 from battery path back to TPS63021 EN pin (signal-level)
- Select C&K OS102011MA1QN1 (100mA SPDT, LCSC C226259), 8.4mm actuator, usable as finger toggle
- Battery always connected, charging while off restored
- Supersedes 2026-08-17 battery-path architecture

New library parts:
- ics:AO3400A (N-ch MOSFET, SOT-23, LCSC C20917)
- passives:0603WAF1000T5E (100ohm 0603, LCSC C22775)
- passives:RC0603JR-074R7L (4.7ohm 0603, LCSC C137621)
- electromech:OS102011MA1QN1 (SPDT slide switch, LCSC C226259)

Docs updated:
- project-log: 3 new entries (display review, power switch reversal, USB hub)
- bom.md: item 25b switch selected, display backlight parts
- block-diagram.md: +BATT net (no switch), U8 EN pin (switched by SW21)
- schematic-completion-plan.md: display sheet LOCKED, section F complete
- task-tracker.md: O2 updated with 2026-08-27 architecture
- ic-by-ic-review.md: Q3 superseded again, DEF-001 updated
- datasheets/README.md: HS20HS072RX pinout verified, SPI confirmed

Generated with [Devin](https://devin.ai)

Co-Authored-By: Devin <158243242+devin-ai-integration[bot]@users.noreply.github.com>
Parts:
- removed C27: 100nF, easyeda2kicad:C0603, symbol passives:CC0603KRX7R9BB104
- removed J_DISP1: 0.5K-HX-12PWB, easyeda2kicad:FPC-SMD_12P-P0.50_HDGC_0.5K-HX-12PWB, symbol connectors:0.5K-HX-12PWB
- removed J_DISP2: 0.5K-HX-8PWB, easyeda2kicad:FPC-SMD_8P-P0.50_HDGC_0.5K-HX-8PWB, symbol connectors:0.5K-HX-8PWB
- removed J_EARPIECE1: S2B-PH-SM4-TB, easyeda2kicad:CONN-SMD_P2.00_S2B-PH-SM4-TB-LF-SN, symbol connectors:S2B-PH-SM4-TB
- removed J_HINGE2: 0.5K-HX-14PWB, easyeda2kicad:FPC-SMD_14P-P0.50_HDGC_0.5K-HX-14PWB, symbol connectors:0.5K-HX-14PWB
- removed R19: 4R7, easyeda2kicad:R0603, symbol passives:RC0603JR-07470RL
Connections:
- no-connect marks 3 -> 0
